File: pcb/6ct-expander/ct_frontend.kicad_sch (KiCad schematic)
At the start: 9 parts, among them J1 SJ-3524-SMT-TR

Commit message: [6CT] Mirror connector pins to match emonPi3 pin out
  - Mirrored to emonPi3 pin out facing *down*
  - Also update board information
Other:
- company: OpenEnergyMonitor / Tilt Ltd (Angus Logan) -> OpenEnergyMonitor / Tilt Ltd
- title: emonPi3 -> emonPi3 / Tx6 6CT expander
Changed lines of the file:
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@@
 	(paper "A4")
 	(title_block
-		(title "emonPi3")
-		(date "2024-03-21")
-		(rev "v0.2")
-		(company "OpenEnergyMonitor / Tilt Ltd (Angus Logan)")
-		(comment 1 "Original design: Trystan Lea & Glynn Hudson")
+		(title "emonPi3 / Tx6 6CT expander")
+		(date "2025-12-10")
+		(rev "v1.1")
+		(company "OpenEnergyMonitor / Tilt Ltd")
+		(comment 1 "Angus Logan, 2025")
 		(comment 2 "Commit hash: gitrev")
 	)
